File: controller_bldc_kicad_Sch_PCB/controller_bldc.kicad_pcb (KiCad board)
At the start: 2 copper layers, 178.1 x 101.9 mm, 55 parts, among them J1 Battery Supply, J2 Emergency Button OUT, J3 Emergency Button IN, J4 Brake, J5 Throttle, J6 LM35, J7 Hall Sensors, J8 Nextion Nx3224T028, J9 BLDC Motor, K1 ADW11, Q1 IRF1010N, Q2 IRF1010N, Q3 IRF1010N, Q4 IRF1010N, Q5 IRF1010N, Q6 IRF1010N, SW1 SW_SPST, SW2 SW_Push, U1 ESP32-DEVKITC-32D, U2 LM317_TO-220, U3 LM7805_TO220, U4 IR2103, U8 IR2103, U9 IR2103

Commit message: PCB v0.5 after autoroute
Routing:
- net +5V: track 0.00 -> 204.4 mm
- net +36V: track 129.6 -> 278.6 mm, vias 0 -> 1
- net Current_Sensor: track 62.4 -> 175.9 mm
- net LM35: track 0.00 -> 77.7 mm
- net Throttle: track 0.00 -> 68.4 mm
- net +12V: track 0.00 -> 67.5 mm
- net TX-LCD: track 0.00 -> 63.0 mm
- net PH2: track 78.3 -> 140.1 mm, vias 0 -> 1
- net HIN3: track 0.00 -> 60.2 mm
- net RX-LCD: track 0.00 -> 58.8 mm
- net PH1: track 82.5 -> 138.2 mm
- net LIN3: track 0.00 -> 55.3 mm
- net PH3: track 74.4 -> 125.5 mm
- net HIN2: track 0.00 -> 48.7 mm
- net LIN2: track 0.00 -> 48.0 mm
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