File: Electrónica y Electromecánica/electeam.sch (KiCad schematic (older format))
At the start: 79 parts, among them J1 Battery after BMS Supply, J2 Hall Sensors, J3 LM35, J4 BLDC Motor, J5 Conn_01x11_Male, Q1 IRF1010N, Q2 IRF1010N, Q3 IRF1010N, Q4 IRF1010N, Q6 IRF1010N, Q7 IRF1010N, SW1 OPC, U1 IR2103, U2 IR2103, U3 Opamp_Dual_Generic, U4 IR2103, U5 LM35-D, U6 ESP32-DEVKITC-32D

Commit message: Just before separating folders and branches According to version independence
Parts:
- U3: value Opamp_Dual_Generic -> AmpOp_Dual_Generic
Connections:
- net Current_Sensor: now also Q?.2 (D); no longer R11.1, R12.2
- net D-IRF1010N: now also Q?.3 (S), R11.1, R12.2; no longer Q?.2 (D), R11.2
- net GND: now also R11.2; no longer Q?.3 (S)
- net Throttle: no longer names the net of R27.2, U6.19 (IO34)
Other:
- note added: "Commutation"
- note added: "Energy System"
- note added: "Low Current"
- moved on the sheet: C1, C10, C11, C12, C13, C2, C3, C4, C5, C6, C7, C8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
