File: Diseño Electrónico/Esquema Global/electeam.sch (KiCad schematic (older format))
At the start: 92 parts, among them J1 Battery after BMS Supply, J2 Hall Sensors, J3 LM35, J4 BLDC Motor, J5 Conn_01x11_Male, Q1 IRF1010N, Q2 IRF1010N, Q3 IRF1010N, Q4 IRF1010N, Q6 IRF1010N, Q7 IRF1010N, SW1 OPC, U1 IR2103, U2 IR2103, U3 AmpOp_Dual_Generic, U4 IR2103, U5 LM35-D, U6 ESP32-DEVKITC-32D

Commit message: Ready to create dev/hotfix branches
Connections:
- net D-IRF1010N renamed S-IRF1010N
Other:
- note added: "Ventilador\nFrenos\nVatímetro\n\nSwitch ON/OFF"
- note removed: "Ventilador\nFrenos\nVatímetro\n\n"
Changed lines of the file:
@@
 $EndComp
 Text GLabel 11400 3950 2    50   Input ~ 0
-D-IRF1010N
+S-IRF1010N
 $Comp
 L Device:R R11
@@
 	12150 8550 12150 8800
 Text GLabel 12150 8800 2    50   Input ~ 0
-D-IRF1010N
+S-IRF1010N
 Wire Wire Line
 	12150 8150 12150 8050
@@
 Pack B+PCB\n
 Text Notes 14750 10200 0    50   ~ 0
-Ventilador\nFrenos\nVatímetro\n\n
+Ventilador\nFrenos\nVatímetro\n\nSwitch ON/OFF
 Text Notes 14700 10800 0    50   ~ 0
 Fix:\nMedir resistencia motor\nMedir inductancia motor\nVerificar si se añade símbolo motor DC\n\n

Commit message: Pending if fan is added or not
Parts:
- added SW1: ON/OFF, symbol Switch:SW_SPST
- added SW3: Freno Mano, symbol Switch:SW_SPST
- SW2: renamed from SW?; value SW_SPST -> Freno de Pie
- gave numbers to parts that had none: 20
- renumbered C10 to C1, C7 to C10, C8 to C11, C9 to C12, C11 to C2, C12 to C3, C2 to C4, C1 to C5, C5 to C6, C3 to C7, C4 to C8, C6 to C9, D7 to D6, D8 to D7, D9 to D8, J2 to J1, J5 to J2, J1 to J5, Q6 to Q7, Q7 to Q8, R3 to R10, R6 to R11, R4 to R12, R5 to R13, R10 to R14, R8 to R18, R9 to R19, R11 to R20, R12 to R21, R13 to R23, R14 to R24, R16 to R25, R17 to R26, R20 to R28, R21 to R29, R22 to R30, R23 to R31, R24 to R32, R25 to R33, R26 to R34, R28 to R35, R15 to R4, R18 to R5, R19 to R6, R29 to R7, R1 to R8, R2 to R9, SW1 to SW4, U3 to U10, U6 to U11, U5 to U4, U1 to U7, U2 to U8, U4 to U9
Connections:
- net +36V: now also SW1.1 (A); no longer D1.1 (K), U2.1 (V+InOut)
- net Brake: now also SW3.1 (A)
- net GND: now also SW3.2 (B)
- new net +36V-SW: D1.1 (K), SW1.2 (B), U2.1 (V+InOut)
Other:
- note added: "Ventilador"
- note removed: "Ventilador\nFrenos\nVatímetro\n\nSwitch ON/OFF"
- moved on the sheet: BT1, SW2, U3
