File: Diseño Electrónico/Esquema y Gerbers PCB/controller_bldc.sch (KiCad schematic (older format))
At the start: 73 parts, among them J1 Battery after BMS Supply, J2 BLDC Motor, J3 Hall Sensors, J4 Conn_01x11_Male, J5 LM35, Q1 IRF1010N, Q2 IRF1010N, Q3 IRF1010N, Q4 IRF1010N, Q5 2N2222, Q6 2N2222, Q7 IRF1010N, Q8 IRF1010N, Q9 IRF1010N, U1 IR2103, U2 IR2103, U3 IR2103, U4 AmpOp_Dual_Generic, U5 ESP32-DEVKITC-32D

Commit message: Pending if fan is added or not
Parts:
- added PS01: LM2596DC-DC, symbol SHARKY:LM2596DC-DC
- added PS02: LM2596DC-DC_copy, symbol SHARKY:LM2596DC-DC_copy
- Q9: footprint Package_TO_SOT_THT_Electeam:TO-220-3_Horizontal_TabDown -> Package_TO_SOT_THT:TO-220-3_Vertical
- R15, R16: footprint Resistor_THT:R_Axial_DIN0207_L6.3mm_D2.5mm_P10.16mm_Horizontal -> (none)
- R17: renamed from R18; footprint Resistor_THT:R_Axial_DIN0207_L6.3mm_D2.5mm_P10.16mm_Horizontal -> (none)
- R22: renamed from R24; footprint Resistor_THT:R_Axial_DIN0207_L6.3mm_D2.5mm_P10.16mm_Horizontal -> (none)
- renumbered C11 to C1, C4 to C10, C5 to C11, C9 to C12, C10 to C13, C12 to C2, C13 to C3, C1 to C4, C6 to C5, C2 to C6, C3 to C9, J3 to J1, J4 to J2, J5 to J3, J2 to J4, J1 to J5, R4 to R10, R2 to R11, R6 to R12, R7 to R13, R9 to R14, R20 to R18, R21 to R19, R5 to R20, R8 to R21, R10 to R23, R11 to R24, R12 to R25, R13 to R26, R14 to R27, R17 to R28, R19 to R29, R22 to R30, R23 to R31, R25 to R32, R26 to R33, R27 to R34, R28 to R35, R29 to R4, R30 to R5, R31 to R6, R32 to R7, R1 to R8, R3 to R9, U4 to U10, U5 to U11, U1 to U7, U2 to U8, U3 to U9
Connections:
- net labels added: +36V-SW, S-IRF1010N
- net labels removed: 36V-Motor, D-IRF1010N, LM2596DC-DC, LM2596DC-DC_copy
- no-connect marks 9 -> 1
Other:
- note added: "PCB"
- moved on the sheet: C1, C10, C11, C12, C13, C2, C3, C4, C5, C6, C7, C8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
